File: OpenFlops.kicad_sch (KiCad schematic)
At the start: 90 parts, among them J99 OSHW_LOGO, P1 FLOPPY_CONN, P10 SD CARD, P11 SD PWR, P12 JUMPER_SD, P2 POWER_INPUT, P3 USB_A_FEMALE, P4 PROG_PORT, P5 JUMPER_JC, P6 ENCODER_PORT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

Commit message: Add files via upload
Connections:
- net GND: no longer U3.2 (PC13), U3.3 (PC14), U3.4 (PC15)
- net ~{rdy_3v3}: now also U1.9

Commit message: Refine design
Parts:
- removed FID1, FID2, FID3: Fiducial, Fiducial:Fiducial_0.75mm_Mask1.5mm, symbol Mechanical:Fiducial
- P12: value JUMPER_SD -> SD_DISABLE
Connections:
- net GND: now also U3.2 (PC13), U3.3 (PC14), U3.4 (PC15)
- net dir: no longer P1.20 (Pin_20), P1.22 (Pin_22), P1.24 (Pin_24), P1.26 (Pin_26), PU6.2, PU7.2, PU8.2, PU9.2, Q2.3 (D), U3.15 (PA1), U3.41 (PA8), U3.62 (PB9)
- new net ~{step}: P1.20 (Pin_20), PU6.2, U3.15 (PA1)
- new net ~{trk0}: P1.26 (Pin_26), PU9.2, Q2.3 (D)
- new net ~{wdata}: P1.22 (Pin_22), PU7.2, U3.41 (PA8)
- new net ~{wgate}: P1.24 (Pin_24), PU8.2, U3.62 (PB9)
Other:
- moved on the sheet: P12
