File: OpenFlops.kicad_sch (KiCad schematic)
At the start: 86 parts, among them P1 FLOPPY_CONN, P10 CONN_SDCARD, P12 SD_DISABLE, P2 POWER_INPUT, P3 USB_A_FEMALE, P4 PROG_PORT, P5 JUMPER_JC, P6 ENCODER_PORT, P7 DISPLAY_PORT, P8 USB_HEADER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

Commit message: Add inversion circuit for SD detect signal
Parts:
- added JP2: JMP_SDCD, Jumper:SolderJumper-3_P1.3mm_Open_RoundedPad1.0x1.5mm, symbol Jumper:Jumper_3_Open
- added Q8: BSS138, Package_TO_SOT_SMD:SOT-23, symbol Transistor_FET:BSS138
- added R8: 1K, Resistor_SMD:R_0805_2012Metric_Pad1.20x1.40mm_HandSolder, symbol Device:R
- added R9: 10k, Resistor_SMD:R_0805_2012Metric_Pad1.20x1.40mm_HandSolder, symbol Device:R
- renumbered P12 to JP1, Q8 to Q4
Connections:
- net +3.3V: now also R9.1
- net GND: now also Q8.2 (S)
- net spi_cd: now also JP2.2 (C); no longer P10.7 (Pin_7)
- new net: Q8.1 (G), R8.1, R9.2
- new net: JP2.3 (B), Q8.3 (D)
- new net ~{spi_cd}: JP2.1 (A), P10.7 (Pin_7), R8.2
Other:
- moved on the sheet: C3, C5, JP1, Y1

Commit message: Make MOSFETs slightly more handsolder-friendly and move Q8 down a bit
Parts:
- Q1, Q2, Q3, Q4, Q5, Q6, Q7, Q8: footprint Package_TO_SOT_SMD:SOT-23 -> OpenFlops:SOT-23_Handsolder
Changed lines of the file:
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@@
 			)
 		)
-		(property "Footprint" "Package_TO_SOT_SMD:SOT-23"
+		(property "Footprint" "OpenFlops:SOT-23_Handsolder"
 			(at 135.89 127.635 0)
 			(effects
@@
 			)
 		)
-		(property "Footprint" "Package_TO_SOT_SMD:SOT-23"
+		(property "Footprint" "OpenFlops:SOT-23_Handsolder"
 			(at 152.4 144.145 0)
 			(effects
@@
 			)
 		)
-		(property "Footprint" "Package_TO_SOT_SMD:SOT-23"
+		(property "Footprint" "OpenFlops:SOT-23_Handsolder"
 			(at 152.4 165.735 0)
 			(effects
@@
 			)
 		)
-		(property "Footprint" "Package_TO_SOT_SMD:SOT-23"
+		(property "Footprint" "OpenFlops:SOT-23_Handsolder"
 			(at 85.09 187.325 0)
 			(effects
@@
 			)
 		)
-		(property "Footprint" "Package_TO_SOT_SMD:SOT-23"
+		(property "Footprint" "OpenFlops:SOT-23_Handsolder"
 			(at 20.32 117.475 0)
 			(effects
@@
 			)
 		)
-		(property "Footprint" "Package_TO_SOT_SMD:SOT-23"
+		(property "Footprint" "OpenFlops:SOT-23_Handsolder"
 			(at 85.09 144.145 0)
 			(effects
@@
 			)
 		)
-		(property "Footprint" "Package_TO_SOT_SMD:SOT-23"
+		(property "Footprint" "OpenFlops:SOT-23_Handsolder"
 			(at 85.09 165.735 0)
 			(effects
@@
 			)
 		)
-		(property "Footprint" "Package_TO_SOT_SMD:SOT-23"
+		(property "Footprint" "OpenFlops:SOT-23_Handsolder"
 			(at 152.4 187.325 0)
 			(effects
